Commit message: include transmission xacro

File: tm_description/urdf/tm700.urdf.xacro (robot description, xacro)
@@ -1,6 +1,8 @@
 <?xml version="1.0"?>
 <robot xmlns:xacro="http://www.ros.org/wiki/xacro">
+  <!-- transmission -->
+  <xacro:include filename="$(find tm_description)/urdf/tm.transmission.xacro" />
+  <!-- Mass parameters -->
   <property name="pi" value="3.14159265" />
-  <!-- Mass parameters-->
   <property name="base_mass" value="1.0" />
   <property name="shoulder_mass" value="4.5" />
@@ -50,4 +52,6 @@
   </xacro:macro>
   <xacro:macro name="tm700_robot" params="prefix joint_limited">
+    <!-- transmission prefix -->
+    <xacro:tm_arm_transmission prefix="${prefix}" />
     <link name="${prefix}base_link" >
       <visual>
@@ -268,6 +272,4 @@
       <origin xyz="0.0 0.0 ${ee_length}" rpy="0.0 0.0 0.0" />
     </joint>
-    <xacro:tm_arm_transmission prefix="${prefix}" />
-    <xacro:tm_arm_gazebo prefix="${prefix}" />
     <!-- ROS base to TM 'base_link' Coordinates transform -->
     <link name="${prefix}base"/>

File: tm_description/urdf/tm700_robot.gazebo.xacro (robot description, xacro)
@@ -1,12 +1,13 @@
 <?xml version="1.0"?>
 <robot name="tm700" xmlns:xacro="http://www.ros.org/wiki/xacro">
-  <!-- gazebo stuff -->
+  <xacro:property name="prefix" value="" />
+  <!-- Gazebo stuff -->
   <xacro:include filename="$(find tm_description)/urdf/common.gazebo.xacro" />
-  <xacro:include filename="$(find tm_description)/urdf/tm.transmission.xacro" />
   <xacro:include filename="$(find tm_description)/urdf/tm.gazebo.xacro" />
+  <xacro:tm_arm_gazebo prefix="${prefix}" />
   <!-- tm700 -->
   <xacro:include filename="$(find tm_description)/urdf/tm700.urdf.xacro" />
   <!-- joint limit -->
-  <xacro:tm700_robot prefix="" joint_limited="false"/>
+  <xacro:tm700_robot prefix="${prefix}" joint_limited="false"/>
   <link name="world" />
   <joint name="world_joint" type="fixed">

File: tm_description/urdf/tm700_robot_joint_limited.gazebo.xacro (robot description, xacro)
@@ -1,12 +1,13 @@
 <?xml version="1.0"?>
 <robot name="tm700" xmlns:xacro="http://www.ros.org/wiki/xacro">
-  <!-- gazebo stuff -->
+  <xacro:property name="prefix" value="" />
+  <!-- Gazebo stuff -->
   <xacro:include filename="$(find tm_description)/urdf/common.gazebo.xacro" />
-  <xacro:include filename="$(find tm_description)/urdf/tm.transmission.xacro" />
   <xacro:include filename="$(find tm_description)/urdf/tm.gazebo.xacro" />
+  <xacro:tm_arm_gazebo prefix="${prefix}" />
   <!-- tm700 -->
   <xacro:include filename="$(find tm_description)/urdf/tm700.urdf.xacro" />
   <!-- joint limit -->
-  <xacro:tm700_robot prefix="" joint_limited="true"/>
+  <xacro:tm700_robot prefix="${prefix}" joint_limited="true"/>
   <link name="world" />
   <joint name="world_joint" type="fixed">
