Commit message: re-run moveit_setup_asistant. delete vitual joint. fix deprecated warnning

File: tm_description/urdf/tm.gazebo.xacro (robot description, xacro)
@@ -2,5 +2,5 @@
 <robot xmlns:xacro="http://www.ros.org/wiki/xacro">
   <xacro:macro name="tm_arm_gazebo" params="prefix">
-    <gazebo reference="${prefix}ase_link">
+    <gazebo reference="${prefix}base_link">
       <selfCollide>true</selfCollide>
     </gazebo>

File: tm_description/urdf/tm700.urdf.xacro (robot description, xacro)
@@ -274,15 +274,15 @@
     <!-- ROS base to TM 'base_link' Coordinates transform -->
     <link name="${prefix}base"/>
-    <joint name="${prefix}base_link-base" type="fixed">
+    <joint name="${prefix}base-base_link" type="fixed">
       <origin xyz="0 0 0" rpy="0 0 0"/>
-      <parent link="${prefix}base_link"/>
-      <child link="${prefix}base"/>
+      <parent link="${prefix}base"/>
+      <child link="${prefix}base_link"/>
     </joint>
     <!-- Frame coincident with all-zeros TCP on TM controller -->
     <link name="${prefix}tool0"/>
-    <joint name="${prefix}last_link-tool0" type="fixed">
-      <parent link="${prefix}wrist_3_link"/>
+    <joint name="${prefix}tip_link-tool0" type="fixed">
+      <parent link="${prefix}tip_link"/>
       <child link="${prefix}tool0"/>
-      <origin xyz="0.0 0.0 ${ee_length}" rpy="0.0 0.0 0.0" />
+      <origin xyz="0 0 0" rpy="0 0 0"/>
     </joint>
   </xacro:macro>

File: tm_description/urdf/tm700_robot.urdf.xacro (robot description, xacro)
@@ -12,5 +12,5 @@
   <joint name="world_joint" type="fixed">
     <parent link="world" />
-    <child link = "base_link" />
+    <child link="base" />
     <origin xyz="0 0 0" rpy="0 0 0" />
   </joint>

File: tm_description/urdf/tm700_robot_eih.urdf.xacro (robot description, xacro)
@@ -12,5 +12,5 @@
   <joint name="world_joint" type="fixed">
     <parent link="world" />
-    <child link = "base_link" />
+    <child link="base" />
     <origin xyz="0 0 0" rpy="0 0 0" />
   </joint>

File: tm_description/urdf/tm700_robot_joint_limited.urdf.xacro (robot description, xacro)
@@ -12,5 +12,5 @@
   <joint name="world_joint" type="fixed">
     <parent link="world" />
-    <child link = "base_link" />
+    <child link="base" />
     <origin xyz="0 0 0" rpy="0 0 0" />
   </joint>

File: tm_description/urdf/tm700_robot_joint_limited_eih.urdf.xacro (robot description, xacro)
@@ -12,5 +12,5 @@
   <joint name="world_joint" type="fixed">
     <parent link="world" />
-    <child link = "base_link" />
+    <child link="base" />
     <origin xyz="0 0 0" rpy="0 0 0" />
   </joint>

File: tm_description/urdf/tm900.urdf.xacro (robot description, xacro)
@@ -273,15 +273,15 @@
     <!-- ROS base to TM 'base_link' Coordinates transform -->
     <link name="${prefix}base"/>
-    <joint name="${prefix}base_link-base" type="fixed">
+    <joint name="${prefix}base-base_link" type="fixed">
       <origin xyz="0 0 0" rpy="0 0 0"/>
-      <parent link="${prefix}base_link"/>
-      <child link="${prefix}base"/>
+      <parent link="${prefix}base"/>
+      <child link="${prefix}base_link"/>
     </joint>
     <!-- Frame coincident with all-zeros TCP on TM controller -->
     <link name="${prefix}tool0"/>
-    <joint name="${prefix}last_link-tool0" type="fixed">
-      <parent link="${prefix}wrist_3_link"/>
+    <joint name="${prefix}tip_link-tool0" type="fixed">
+      <parent link="${prefix}tip_link"/>
       <child link="${prefix}tool0"/>
-      <origin xyz="0.0 0.0 ${ee_length}" rpy="0.0 0.0 0.0" />
+      <origin xyz="0 0 0" rpy="0 0 0"/>
     </joint>
   </xacro:macro>

File: tm_description/urdf/tm900_robot.urdf.xacro (robot description, xacro)
@@ -12,5 +12,5 @@
   <joint name="world_joint" type="fixed">
     <parent link="world" />
-    <child link = "base_link" />
+    <child link="base" />
     <origin xyz="0 0 0" rpy="0 0 0" />
   </joint>

File: tm_description/urdf/tm900_robot_eih.urdf.xacro (robot description, xacro)
@@ -12,5 +12,5 @@
   <joint name="world_joint" type="fixed">
     <parent link="world" />
-    <child link = "base_link" />
+    <child link="base" />
     <origin xyz="0 0 0" rpy="0 0 0" />
   </joint>

File: tm_description/urdf/tm900_robot_joint_limited.urdf.xacro (robot description, xacro)
@@ -12,5 +12,5 @@
   <joint name="world_joint" type="fixed">
     <parent link="world" />
-    <child link = "base_link" />
+    <child link="base" />
     <origin xyz="0 0 0" rpy="0 0 0" />
   </joint>

File: tm_description/urdf/tm900_robot_joint_limited_eih.urdf.xacro (robot description, xacro)
@@ -12,5 +12,5 @@
   <joint name="world_joint" type="fixed">
     <parent link="world" />
-    <child link = "base_link" />
+    <child link="base" />
     <origin xyz="0 0 0" rpy="0 0 0" />
   </joint>
