Commit message: gazebo eye-in-hand camera simulation

File: tm_description/urdf/common.gazebo.xacro (robot description, xacro)
@@ -2,9 +2,9 @@
 <robot xmlns:xacro="http://www.ros.org/wiki/xacro">
   <gazebo>
-    <plugin name="ros_control" filename="libgazebo_ros_control.so">
+    <plugin name="gazebo_ros_control" filename="libgazebo_ros_control.so">
       <!--robotNamespace>/</robotNamespace-->
       <!--robotSimType>gazebo_ros_control/DefaultRobotHWSim</robotSimType-->
     </plugin>
-<!--
+    <!--
     <plugin name="gazebo_ros_power_monitor_controller" filename="libgazebo_ros_power_monitor.so">
       <alwaysOn>true</alwaysOn>
@@ -19,5 +19,5 @@
       <chargeVoltage>16.41</chargeVoltage>
     </plugin>
--->
+    -->
   </gazebo>
 </robot>

File: tm_description/urdf/tm.gazebo.xacro (robot description, xacro)
@@ -2,5 +2,25 @@
 <robot xmlns:xacro="http://www.ros.org/wiki/xacro">
   <xacro:macro name="tm_arm_gazebo" params="prefix">
-    <!-- nothing to do here at the moment -->
+    <gazebo reference="${prefix}ase_link">
+      <selfCollide>true</selfCollide>
+    </gazebo>
+    <gazebo reference="${prefix}shoulder_1_link">
+      <selfCollide>true</selfCollide>
+    </gazebo>
+    <gazebo reference="${prefix}arm_1_link">
+      <selfCollide>true</selfCollide>
+    </gazebo>
+    <gazebo reference="${prefix}arm_2_link">
+      <selfCollide>true</selfCollide>
+    </gazebo>
+    <gazebo reference="${prefix}wrist_1_link">
+      <selfCollide>true</selfCollide>
+    </gazebo>
+    <gazebo reference="${prefix}wrist_2_link">
+      <selfCollide>true</selfCollide>
+    </gazebo>
+    <gazebo reference="${prefix}wrist_3_link">
+      <selfCollide>true</selfCollide>
+    </gazebo>
   </xacro:macro>
 </robot>

File: tm_description/urdf/tm700_robot.urdf.xacro (robot description, xacro)
@@ -1,13 +1,17 @@
 <?xml version="1.0"?>
 <robot name="tm700" xmlns:xacro="http://www.ros.org/wiki/xacro">
+  <xacro:property name="prefix" value="" />
+  <!-- gazebo stuff -->
+  <xacro:include filename="$(find tm_description)/urdf/common.gazebo.xacro" />
+  <xacro:include filename="$(find tm_description)/urdf/tm.gazebo.xacro" />
+  <xacro:tm_arm_gazebo prefix="${prefix}" />
   <!-- tm700 -->
   <xacro:include filename="$(find tm_description)/urdf/tm700.urdf.xacro" />
-  <!-- arm -->
-  <xacro:tm700_robot prefix="" joint_limited="false"/>
+  <xacro:tm700_robot prefix="${prefix}" joint_limited="false" />
   <link name="world" />
   <joint name="world_joint" type="fixed">
     <parent link="world" />
     <child link = "base_link" />
-    <origin xyz="0.0 0.0 0.0" rpy="0.0 0.0 0.0" />
+    <origin xyz="0 0 0" rpy="0 0 0" />
   </joint>
 </robot>

File: tm_description/urdf/tm700_robot_eih.urdf.xacro (robot description, xacro)
@@ -2,5 +2,5 @@
 <robot name="tm700" xmlns:xacro="http://www.ros.org/wiki/xacro">
   <xacro:property name="prefix" value="" />
-  <!-- Gazebo stuff -->
+  <!-- gazebo stuff -->
   <xacro:include filename="$(find tm_description)/urdf/common.gazebo.xacro" />
   <xacro:include filename="$(find tm_description)/urdf/tm.gazebo.xacro" />
@@ -8,11 +8,13 @@
   <!-- tm700 -->
   <xacro:include filename="$(find tm_description)/urdf/tm700.urdf.xacro" />
-  <!-- joint limit -->
-  <xacro:tm700_robot prefix="${prefix}" joint_limited="false"/>
+  <xacro:tm700_robot prefix="${prefix}" joint_limited="false" />
   <link name="world" />
   <joint name="world_joint" type="fixed">
     <parent link="world" />
     <child link = "base_link" />
-    <origin xyz="0.0 0.0 0.0" rpy="0.0 0.0 0.0" />
+    <origin xyz="0 0 0" rpy="0 0 0" />
   </joint>
+  <!-- eye in hand camera-->
+  <xacro:include filename="$(find tm_description)/urdf/tm700.eih.xacro" />
+  <xacro:tm700_eih_camera prefix="${prefix}" />
 </robot>

File: tm_description/urdf/tm700_robot_joint_limited_eih.urdf.xacro (robot description, xacro)
@@ -2,5 +2,5 @@
 <robot name="tm700" xmlns:xacro="http://www.ros.org/wiki/xacro">
   <xacro:property name="prefix" value="" />
-  <!-- Gazebo stuff -->
+  <!-- gazebo stuff -->
   <xacro:include filename="$(find tm_description)/urdf/common.gazebo.xacro" />
   <xacro:include filename="$(find tm_description)/urdf/tm.gazebo.xacro" />
@@ -8,11 +8,13 @@
   <!-- tm700 -->
   <xacro:include filename="$(find tm_description)/urdf/tm700.urdf.xacro" />
-  <!-- joint limit -->
-  <xacro:tm700_robot prefix="${prefix}" joint_limited="true"/>
+  <xacro:tm700_robot prefix="${prefix}" joint_limited="true" />
   <link name="world" />
   <joint name="world_joint" type="fixed">
     <parent link="world" />
     <child link = "base_link" />
-    <origin xyz="0.0 0.0 0.0" rpy="0.0 0.0 0.0" />
+    <origin xyz="0 0 0" rpy="0 0 0" />
   </joint>
+  <!-- eye in hand camera-->
+  <xacro:include filename="$(find tm_description)/urdf/tm700.eih.xacro" />
+  <xacro:tm700_eih_camera prefix="${prefix}" />
 </robot>

File: tm_description/urdf/tm900.urdf.xacro (robot description, xacro)
@@ -2,5 +2,4 @@
 <robot xmlns:xacro="http://www.ros.org/wiki/xacro">
   <xacro:include filename="$(find tm_description)/urdf/tm.transmission.xacro" />
-  <xacro:include filename="$(find tm_description)/urdf/tm.gazebo.xacro" />
   <property name="pi" value="3.14159265" />
   <!-- Mass parameters-->
@@ -52,4 +51,6 @@
   </xacro:macro>
   <xacro:macro name="tm900_robot" params="prefix joint_limited">
+    <!-- transmission prefix -->
+    <xacro:tm_arm_transmission prefix="${prefix}" />
     <link name="${prefix}base_link" >
       <visual>
@@ -270,6 +271,4 @@
       <origin xyz="0.0 0.0 ${ee_length}" rpy="0.0 0.0 0.0" />
     </joint>
-    <xacro:tm_arm_transmission prefix="${prefix}" />
-    <xacro:tm_arm_gazebo prefix="${prefix}" />
     <!-- ROS base to TM 'base_link' Coordinates transform -->
     <link name="${prefix}base"/>

File: tm_description/urdf/tm900_robot.urdf.xacro (robot description, xacro)
@@ -1,15 +1,17 @@
 <?xml version="1.0"?>
 <robot name="tm900" xmlns:xacro="http://www.ros.org/wiki/xacro">
-  <!-- common stuff -->
+  <xacro:property name="prefix" value="" />
+  <!-- gazebo stuff -->
   <xacro:include filename="$(find tm_description)/urdf/common.gazebo.xacro" />
+  <xacro:include filename="$(find tm_description)/urdf/tm.gazebo.xacro" />
+  <xacro:tm_arm_gazebo prefix="${prefix}" />
   <!-- tm900 -->
   <xacro:include filename="$(find tm_description)/urdf/tm900.urdf.xacro" />
-  <!-- arm -->
-  <xacro:tm900_robot prefix="" joint_limited="false"/>
+  <xacro:tm900_robot prefix="${prefix}" joint_limited="false" />
   <link name="world" />
   <joint name="world_joint" type="fixed">
     <parent link="world" />
     <child link = "base_link" />
-    <origin xyz="0.0 0.0 0.0" rpy="0.0 0.0 0.0" />
+    <origin xyz="0 0 0" rpy="0 0 0" />
   </joint>
 </robot>

File: tm_description/urdf/tm900_robot_eih.urdf.xacro (robot description, xacro)
@@ -1,4 +1,4 @@
 <?xml version="1.0"?>
-<robot name="tm700" xmlns:xacro="http://www.ros.org/wiki/xacro">
+<robot name="tm900" xmlns:xacro="http://www.ros.org/wiki/xacro">
   <xacro:property name="prefix" value="" />
   <!-- gazebo stuff -->
@@ -6,7 +6,7 @@
   <xacro:include filename="$(find tm_description)/urdf/tm.gazebo.xacro" />
   <xacro:tm_arm_gazebo prefix="${prefix}" />
-  <!-- tm700 -->
-  <xacro:include filename="$(find tm_description)/urdf/tm700.urdf.xacro" />
-  <xacro:tm700_robot prefix="${prefix}" joint_limited="true" />
+  <!-- tm900 -->
+  <xacro:include filename="$(find tm_description)/urdf/tm900.urdf.xacro" />
+  <xacro:tm900_robot prefix="${prefix}" joint_limited="false" />
   <link name="world" />
   <joint name="world_joint" type="fixed">
@@ -15,3 +15,6 @@
     <origin xyz="0 0 0" rpy="0 0 0" />
   </joint>
+  <!-- eye in hand camera-->
+  <xacro:include filename="$(find tm_description)/urdf/tm900.eih.xacro" />
+  <xacro:tm900_eih_camera prefix="${prefix}" />
 </robot>

File: tm_description/urdf/tm900_robot_joint_limited.urdf.xacro (robot description, xacro)
@@ -1,15 +1,17 @@
 <?xml version="1.0"?>
 <robot name="tm900" xmlns:xacro="http://www.ros.org/wiki/xacro">
-  <!-- common stuff -->
+  <xacro:property name="prefix" value="" />
+  <!-- gazebo stuff -->
   <xacro:include filename="$(find tm_description)/urdf/common.gazebo.xacro" />
+  <xacro:include filename="$(find tm_description)/urdf/tm.gazebo.xacro" />
+  <xacro:tm_arm_gazebo prefix="${prefix}" />
   <!-- tm900 -->
   <xacro:include filename="$(find tm_description)/urdf/tm900.urdf.xacro" />
-  <!-- arm -->
-  <xacro:tm700_robot prefix="" joint_limited="true"/>
+  <xacro:tm900_robot prefix="${prefix}" joint_limited="true" />
   <link name="world" />
   <joint name="world_joint" type="fixed">
     <parent link="world" />
     <child link = "base_link" />
-    <origin xyz="0.0 0.0 0.0" rpy="0.0 0.0 0.0" />
+    <origin xyz="0 0 0" rpy="0 0 0" />
   </joint>
 </robot>

File: tm_description/urdf/tm900_robot_joint_limited_eih.urdf.xacro (robot description, xacro)
@@ -1,4 +1,4 @@
 <?xml version="1.0"?>
-<robot name="tm700" xmlns:xacro="http://www.ros.org/wiki/xacro">
+<robot name="tm900" xmlns:xacro="http://www.ros.org/wiki/xacro">
   <xacro:property name="prefix" value="" />
   <!-- gazebo stuff -->
@@ -6,7 +6,7 @@
   <xacro:include filename="$(find tm_description)/urdf/tm.gazebo.xacro" />
   <xacro:tm_arm_gazebo prefix="${prefix}" />
-  <!-- tm700 -->
-  <xacro:include filename="$(find tm_description)/urdf/tm700.urdf.xacro" />
-  <xacro:tm700_robot prefix="${prefix}" joint_limited="true" />
+  <!-- tm900 -->
+  <xacro:include filename="$(find tm_description)/urdf/tm900.urdf.xacro" />
+  <xacro:tm900_robot prefix="${prefix}" joint_limited="true" />
   <link name="world" />
   <joint name="world_joint" type="fixed">
@@ -15,3 +15,6 @@
     <origin xyz="0 0 0" rpy="0 0 0" />
   </joint>
+  <!-- eye in hand camera-->
+  <xacro:include filename="$(find tm_description)/urdf/tm900.eih.xacro" />
+  <xacro:tm900_eih_camera prefix="${prefix}" />
 </robot>
