Commit message: 1100, 1300 add

File: tm_description/urdf/common.gazebo.xacro (robot description, xacro)
@@ -5,4 +5,5 @@
       <!--robotNamespace>/</robotNamespace-->
       <!--robotSimType>gazebo_ros_control/DefaultRobotHWSim</robotSimType-->
+      <legacyModeNS>true</legacyModeNS>
     </plugin>
     <!--

File: tm_description/urdf/tm.transmission.xacro (robot description, xacro)
@@ -5,5 +5,5 @@
       <type>transmission_interface/SimpleTransmission</type>
       <joint name="${prefix}shoulder_1_joint">
-        <hardwareInterface>PositionJointInterface</hardwareInterface>
+        <hardwareInterface>hardware_interface/PositionJointInterface</hardwareInterface>
       </joint>
       <actuator name="${prefix}shoulder_1_motor">
@@ -14,5 +14,5 @@
       <type>transmission_interface/SimpleTransmission</type>
       <joint name="${prefix}shoulder_2_joint">
-        <hardwareInterface>PositionJointInterface</hardwareInterface>
+        <hardwareInterface>hardware_interface/PositionJointInterface</hardwareInterface>
       </joint>
       <actuator name="${prefix}shoulder_2_motor">
@@ -23,5 +23,5 @@
       <type>transmission_interface/SimpleTransmission</type>
       <joint name="${prefix}elbow_1_joint">
-        <hardwareInterface>PositionJointInterface</hardwareInterface>
+        <hardwareInterface>hardware_interface/PositionJointInterface</hardwareInterface>
       </joint>
       <actuator name="${prefix}elbow_1_motor">
@@ -32,5 +32,5 @@
       <type>transmission_interface/SimpleTransmission</type>
       <joint name="${prefix}wrist_1_joint">
-        <hardwareInterface>PositionJointInterface</hardwareInterface>
+        <hardwareInterface>hardware_interface/PositionJointInterface</hardwareInterface>
       </joint>
       <actuator name="${prefix}wrist_1_motor">
@@ -41,5 +41,5 @@
       <type>transmission_interface/SimpleTransmission</type>
       <joint name="${prefix}wrist_2_joint">
-        <hardwareInterface>PositionJointInterface</hardwareInterface>
+        <hardwareInterface>hardware_interface/PositionJointInterface</hardwareInterface>
       </joint>
       <actuator name="${prefix}wrist_2_motor">
@@ -50,5 +50,5 @@
       <type>transmission_interface/SimpleTransmission</type>
       <joint name="${prefix}wrist_3_joint">
-        <hardwareInterface>PositionJointInterface</hardwareInterface>
+        <hardwareInterface>hardware_interface/PositionJointInterface</hardwareInterface>
       </joint>
       <actuator name="${prefix}wrist_3_motor">

File: tm_description/urdf/tm1100.urdf.xacro (robot description, xacro)
@@ -4,12 +4,11 @@
   <xacro:include filename="$(find tm_description)/urdf/tm.transmission.xacro" />
   <!-- Mass parameters -->
-  <property name="pi" value="3.14159265" />
-  <property name="base_mass" value="1.0" />
-  <property name="shoulder_mass" value="4.5" />
-  <property name="arm_1_mass" value="10.5" />
-  <property name="arm_2_mass" value="2.1" />
-  <property name="wrist_1_mass" value="1.45" />
-  <property name="wrist_2_mass" value="1.45" />
-  <property name="wrist_3_mass" value="0.4" />
+  <xacro:property name="base_mass" value="1.0" />
+  <xacro:property name="shoulder_mass" value="4.5" />
+  <xacro:property name="arm_1_mass" value="10.5" />
+  <xacro:property name="arm_2_mass" value="2.1" />
+  <xacro:property name="wrist_1_mass" value="1.45" />
+  <xacro:property name="wrist_2_mass" value="1.45" />
+  <xacro:property name="wrist_3_mass" value="0.4" />
   <!-- Kinematic model -->
   <!-- Properties from tmcontrol.conf -->
@@ -24,26 +23,26 @@
     center_of_mass = [ [0, -0.02561, 0.00193], [0.2125, 0, 0.11336], [0.11993, 0.0, 0.0265], [0, -0.0018, 0.01634], [0, 0.0018,0.01634], [0, 0, -0.001159] ]
   -->
-  <property name="tm_d1" value="0.1652" />
-  <property name="tm_a2" value="0.5361" />
-  <property name="tm_a3" value="0.4579" />
-  <property name="tm_d4" value="0.1563" />
-  <property name="tm_d5" value="0.1060" />
-  <property name="tm_d6" value="0.11315" />
+  <xacro:property name="tm_d1" value="0.1652" />
+  <xacro:property name="tm_a2" value="0.5361" />
+  <xacro:property name="tm_a3" value="0.4579" />
+  <xacro:property name="tm_d4" value="0.1563" />
+  <xacro:property name="tm_d5" value="0.1060" />
+  <xacro:property name="tm_d6" value="0.11315" />
   <!-- offsets for shoulder/elbow joints -->
-  <property name="shoulder_offset" value="-0.1801" />  <!-- measured from model -->
-  <property name="elbow_offset" value="0.1298" /> <!-- measured from model -->
-  <property name="wrist_offset" value="${-tm_d4 - elbow_offset - shoulder_offset}" />
+  <xacro:property name="shoulder_offset" value="-0.1801" />  <!-- measured from model -->
+  <xacro:property name="elbow_offset" value="0.1298" /> <!-- measured from model -->
+  <xacro:property name="wrist_offset" value="${-tm_d4 - elbow_offset - shoulder_offset}" />
   <!-- link lengths used in model -->
-  <property name="shoulder_height" value="${tm_d1}" />
-  <property name="arm_1_length" value="${tm_a2}" />
-  <property name="arm_2_length" value="${tm_a3}" />
-  <property name="wrist_1_length" value="tm_d5}" />
-  <property name="wrist_2_length" value="${tm_d5}" />
-  <property name="wrist_3_length" value="0.05525" />
-  <property name="ee_length" value="${tm_d6 - wrist_3_length}" />
+  <xacro:property name="shoulder_height" value="${tm_d1}" />
+  <xacro:property name="arm_1_length" value="${tm_a2}" />
+  <xacro:property name="arm_2_length" value="${tm_a3}" />
+  <xacro:property name="wrist_1_length" value="tm_d5}" />
+  <xacro:property name="wrist_2_length" value="${tm_d5}" />
+  <xacro:property name="wrist_3_length" value="0.05525" />
+  <xacro:property name="ee_length" value="${tm_d6 - wrist_3_length}" />
   <xacro:macro name="cylinder_inertial" params="radius length mass *origin">
     <inertial>
       <mass value="${mass}" />
-      <insert_block name="origin" />
+      <xacro:insert_block name="origin" />
       <inertia ixx="${0.0833333 * mass * (3 * radius * radius + length * length)}" ixy="0.0" ixz="0.0"
         iyy="${0.0833333 * mass * (3 * radius * radius + length * length)}" iyz="0.0"
@@ -51,5 +50,5 @@
     </inertial>
   </xacro:macro>
-  <xacro:macro name="tm1100_robot" params="prefix joint_limited">
+  <xacro:macro name="tm1100_robot" params="prefix joint_limited has_camera">
     <!-- transmission prefix -->
     <xacro:tm_arm_transmission prefix="${prefix}" />
@@ -96,8 +95,8 @@
       <axis xyz="0 -1 0" />
       <xacro:unless value="${joint_limited}">
-        <limit lower="${-2.0 * pi}" upper="${2.0 * pi}" effort="150.0" velocity="3.15"/>
-      </xacro:unless>
-      <xacro:if value="${joint_limited}">
-        <limit lower="${-pi}" upper="${pi}" effort="150.0" velocity="3.15"/>
+        <limit lower="${-270. / 180. * pi}" upper="${270. / 180. * pi}" effort="150.0" velocity="${120. / 180. * pi}"/>
+      </xacro:unless>
+      <xacro:if value="${joint_limited}">
+        <limit lower="${-pi}" upper="${pi}" effort="150.0" velocity="${120. / 180. * pi}"/>
       </xacro:if>
       <dynamics damping="0.0" friction="0.0"/>
@@ -127,8 +126,8 @@
       <axis xyz="0 0 1" />
       <xacro:unless value="${joint_limited}">
-        <limit lower="${-1.5 * pi}" upper="${1.5 * pi}" effort="150.0" velocity="3.15"/>
-      </xacro:unless>
-      <xacro:if value="${joint_limited}">
-        <limit lower="${-pi}" upper="${pi}" effort="150.0" velocity="3.15"/>
+        <limit lower="${-180. / 180. * pi}" upper="${180. / 180. * pi}" effort="150.0" velocity="${120. / 180. * pi}"/>
+      </xacro:unless>
+      <xacro:if value="${joint_limited}">
+        <limit lower="${-pi}" upper="${pi}" effort="150.0" velocity="${120. / 180. * pi}"/>
       </xacro:if>
       <dynamics damping="0.0" friction="0.0"/>
@@ -158,8 +157,8 @@
       <axis xyz="0 0 1" />
       <xacro:unless value="${joint_limited}">
-        <limit lower="${-1.5 * pi}" upper="${1.5 * pi}" effort="150.0" velocity="3.15"/>
-      </xacro:unless>
-      <xacro:if value="${joint_limited}">
-        <limit lower="${-pi}" upper="${pi}" effort="150.0" velocity="3.15"/>
+        <limit lower="${-163. / 180. * pi}" upper="${163. / 180. * pi}" effort="150.0" velocity="${150. / 180. * pi}"/>
+      </xacro:unless>
+      <xacro:if value="${joint_limited}">
+        <limit lower="${-pi}" upper="${pi}" effort="150.0" velocity="${180. / 180. * pi}"/>
       </xacro:if>
       <dynamics damping="0.0" friction="0.0"/>
@@ -189,8 +188,8 @@
       <axis xyz="0 1 0" />
       <xacro:unless value="${joint_limited}">
-        <limit lower="${-2.0 * pi}" upper="${2.0 * pi}" effort="28.0" velocity="3.2"/>
-      </xacro:unless>
-      <xacro:if value="${joint_limited}">
-        <limit lower="${-pi}" upper="${pi}" effort="28.0" velocity="3.2"/>
+        <limit lower="${-180. / 180. * pi}" upper="${180. / 180. * pi}" effort="28.0" velocity="${180. / 180. * pi}"/>
+      </xacro:unless>
+      <xacro:if value="${joint_limited}">
+        <limit lower="${-pi}" upper="${pi}" effort="28.0" velocity="${180. / 180. * pi}"/>
       </xacro:if>
       <dynamics damping="0.0" friction="0.0"/>
@@ -220,8 +219,8 @@
       <axis xyz="0 1 0" />
       <xacro:unless value="${joint_limited}">
-        <limit lower="${-2.0 * pi}" upper="${2.0 * pi}" effort="28.0" velocity="3.2"/>
-      </xacro:unless>
-      <xacro:if value="${joint_limited}">
-        <limit lower="${-pi}" upper="${pi}" effort="28.0" velocity="3.2"/>
+        <limit lower="${-180. / 180. * pi}" upper="${180. / 180. * pi}" effort="28.0" velocity="${180. / 180. * pi}"/>
+      </xacro:unless>
+      <xacro:if value="${joint_limited}">
+        <limit lower="${-pi}" upper="${pi}" effort="28.0" velocity="${180. / 180. * pi}"/>
       </xacro:if>
       <dynamics damping="0.0" friction="0.0"/>
@@ -230,5 +229,10 @@
       <visual>
         <geometry>
-	  <mesh filename="package://tm_description/meshes/tm1100/visual/Wrist3.STL" />
+          <xacro:if value="${has_camera}">
+          <mesh filename="package://tm_description/meshes/tm1100/visual/Wrist3.STL" />
+          </xacro:if>
+          <xacro:unless value="${has_camera}">
+          <mesh filename="package://tm_description/meshes/tm1100/visual/Wrist3_no_camera.STL" />
+          </xacro:unless>
         </geometry>
 	<origin xyz="0 0 0.015" rpy="0 0 0"/>
@@ -239,5 +243,10 @@
       <collision>
         <geometry>
-	  <mesh filename="package://tm_description/meshes/tm1100/collision/wrist_3.STL" />
+          <xacro:if value="${has_camera}">
+	      <mesh filename="package://tm_description/meshes/tm1100/collision/wrist_3.STL" />
+          </xacro:if>
+          <xacro:unless value="${has_camera}">
+	      <mesh filename="package://tm_description/meshes/tm1100/collision/wrist_3_no_camera.STL" />
+          </xacro:unless>
         </geometry>
       </collision>
@@ -252,8 +261,8 @@
       <axis xyz="0 0 1" />
       <xacro:unless value="${joint_limited}">
-        <limit lower="${-2.0 * pi}" upper="${2.0 * pi}" effort="28.0" velocity="3.2"/>
-      </xacro:unless>
-      <xacro:if value="${joint_limited}">
-        <limit lower="${-pi}" upper="${pi}" effort="28.0" velocity="3.2"/>
+        <limit lower="${-270. / 180. * pi}" upper="${270. / 180. * pi}" effort="28.0" velocity="${180. / 180. * pi}"/>
+      </xacro:unless>
+      <xacro:if value="${joint_limited}">
+        <limit lower="${-pi}" upper="${pi}" effort="28.0" velocity="${180. / 180. * pi}"/>
       </xacro:if>
       <dynamics damping="0.0" friction="0.0"/>
@@ -276,6 +285,6 @@
     <joint name="${prefix}base-base_link" type="fixed">
       <origin xyz="0 0 0" rpy="0 0 0"/>
-      <parent link="${prefix}base"/>
-      <child link="${prefix}base_link"/>
+      <parent link="${prefix}base_link"/>
+      <child link="${prefix}base"/>
     </joint>
     <!-- Frame coincident with all-zeros TCP on TM controller -->

File: tm_description/urdf/tm700.urdf.xacro (robot description, xacro)
@@ -4,12 +4,11 @@
   <xacro:include filename="$(find tm_description)/urdf/tm.transmission.xacro" />
   <!-- Mass parameters -->
-  <property name="pi" value="3.14159265" />
-  <property name="base_mass" value="1.0" />
-  <property name="shoulder_mass" value="4.5" />
-  <property name="arm_1_mass" value="10.5" />
-  <property name="arm_2_mass" value="2.1" />
-  <property name="wrist_1_mass" value="1.45" />
-  <property name="wrist_2_mass" value="1.45" />
-  <property name="wrist_3_mass" value="0.4" />
+  <xacro:property name="base_mass" value="1.0" />
+  <xacro:property name="shoulder_mass" value="4.5" />
+  <xacro:property name="arm_1_mass" value="10.5" />
+  <xacro:property name="arm_2_mass" value="2.1" />
+  <xacro:property name="wrist_1_mass" value="1.45" />
+  <xacro:property name="wrist_2_mass" value="1.45" />
+  <xacro:property name="wrist_3_mass" value="0.4" />
   <!-- Kinematic model -->
   <!-- Properties from tmcontrol.conf -->
@@ -24,26 +23,26 @@
     center_of_mass = [ [0, -0.02561, 0.00193], [0.2125, 0, 0.11336], [0.11993, 0.0, 0.0265], [0, -0.0018, 0.01634], [0, 0.0018,0.01634], [0, 0, -0.001159] ](tm700)
   -->
-  <property name="tm_d1" value="0.1451" />
-  <property name="tm_a2" value="0.3290" />
-  <property name="tm_a3" value="0.3115" />
-  <property name="tm_d4" value="0.1222" />
-  <property name="tm_d5" value="0.1060" />
-  <property name="tm_d6" value="0.1144" />
+  <xacro:property name="tm_d1" value="0.1451" />
+  <xacro:property name="tm_a2" value="0.3290" />
+  <xacro:property name="tm_a3" value="0.3115" />
+  <xacro:property name="tm_d4" value="0.1222" />
+  <xacro:property name="tm_d5" value="0.1060" />
+  <xacro:property name="tm_d6" value="0.1144" />
   <!-- offsets for shoulder/elbow joints -->
-  <property name="shoulder_offset" value="-0.146" />  <!-- measured from model -->
-  <property name="elbow_offset" value="0.1298" /> <!-- measured from model -->
-  <property name="wrist_offset" value="${-tm_d4 - elbow_offset - shoulder_offset}" />
+  <xacro:property name="shoulder_offset" value="-0.146" />  <!-- measured from model -->
+  <xacro:property name="elbow_offset" value="0.1298" /> <!-- measured from model -->
+  <xacro:property name="wrist_offset" value="${-tm_d4 - elbow_offset - shoulder_offset}" />
   <!-- link lengths used in model -->
-  <property name="shoulder_height" value="${tm_d1}" />
-  <property name="arm_1_length" value="${tm_a2}" />
-  <property name="arm_2_length" value="${tm_a3}" />
-  <property name="wrist_1_length" value="tm_d5}" />
-  <property name="wrist_2_length" value="${tm_d5}" />
-  <property name="wrist_3_length" value="0.0565" />
-  <property name="ee_length" value="${tm_d6 - wrist_3_length}" />
+  <xacro:property name="shoulder_height" value="${tm_d1}" />
+  <xacro:property name="arm_1_length" value="${tm_a2}" />
+  <xacro:property name="arm_2_length" value="${tm_a3}" />
+  <xacro:property name="wrist_1_length" value="tm_d5}" />
+  <xacro:property name="wrist_2_length" value="${tm_d5}" />
+  <xacro:property name="wrist_3_length" value="0.0565" />
+  <xacro:property name="ee_length" value="${tm_d6 - wrist_3_length}" />
   <xacro:macro name="cylinder_inertial" params="radius length mass *origin">
     <inertial>
       <mass value="${mass}" />
-      <insert_block name="origin" />
+      <xacro:insert_block name="origin" />
       <inertia ixx="${0.0833333 * mass * (3 * radius * radius + length * length)}" ixy="0.0" ixz="0.0"
         iyy="${0.0833333 * mass * (3 * radius * radius + length * length)}" iyz="0.0"
@@ -51,5 +50,5 @@
     </inertial>
   </xacro:macro>
-  <xacro:macro name="tm700_robot" params="prefix joint_limited">
+  <xacro:macro name="tm700_robot" params="prefix joint_limited has_camera">
     <!-- transmission prefix -->
     <xacro:tm_arm_transmission prefix="${prefix}" />
@@ -96,8 +95,8 @@
       <axis xyz="0 -1 0" />
       <xacro:unless value="${joint_limited}">
-        <limit lower="${-2.0 * pi}" upper="${2.0 * pi}" effort="150.0" velocity="3.15"/>
-      </xacro:unless>
-      <xacro:if value="${joint_limited}">
-        <limit lower="${-pi}" upper="${pi}" effort="150.0" velocity="3.15"/>
+        <limit lower="${-270. / 180. * pi}" upper="${270. / 180. * pi}" effort="150.0" velocity="${180 / 180. * pi}"/>
+      </xacro:unless>
+      <xacro:if value="${joint_limited}">
+        <limit lower="${-pi}" upper="${pi}" effort="150.0" velocity="${180 / 180. * pi}"/>
       </xacro:if>
       <dynamics damping="0.0" friction="0.0"/>
@@ -127,8 +126,8 @@
       <axis xyz="0 0 1" />
       <xacro:unless value="${joint_limited}">
-        <limit lower="${-1.5 * pi}" upper="${1.5 * pi}" effort="150.0" velocity="3.15"/>
-      </xacro:unless>
-      <xacro:if value="${joint_limited}">
-        <limit lower="${-pi}" upper="${pi}" effort="150.0" velocity="3.15"/>
+        <limit lower="${-180. / 180. * pi}" upper="${180. / 180. * pi}" effort="150.0" velocity="${180 / 180. * pi}"/>
+      </xacro:unless>
+      <xacro:if value="${joint_limited}">
+        <limit lower="${-pi}" upper="${pi}" effort="150.0" velocity="${180 / 180. * pi}"/>
       </xacro:if>
       <dynamics damping="0.0" friction="0.0"/>
@@ -157,10 +156,5 @@
       <origin xyz="${arm_1_length} 0.0 ${elbow_offset}" rpy="0.0 0.0 0.0" />
       <axis xyz="0 0 1" />
-      <xacro:unless value="${joint_limited}">
-        <limit lower="${-1.5 * pi}" upper="${1.5 * pi}" effort="150.0" velocity="3.15"/>
-      </xacro:unless>
-      <xacro:if value="${joint_limited}">
-        <limit lower="${-pi}" upper="${pi}" effort="150.0" velocity="3.15"/>
-      </xacro:if>
+      <limit lower="${-155. / 180. * pi}" upper="${155. / 180. * pi}" effort="150.0" velocity="${180 / 180. * pi}"/>
       <dynamics damping="0.0" friction="0.0"/>
     </joint>
@@ -189,8 +183,8 @@
       <axis xyz="0 1 0" />
       <xacro:unless value="${joint_limited}">
-        <limit lower="${-2.0 * pi}" upper="${2.0 * pi}" effort="28.0" velocity="3.2"/>
-      </xacro:unless>
-      <xacro:if value="${joint_limited}">
-        <limit lower="${-pi}" upper="${pi}" effort="28.0" velocity="3.2"/>
+        <limit lower="${-180. / 180. * pi}" upper="${180. / 180. * pi}" effort="28.0" velocity="${225. / 180. * pi}"/>
+      </xacro:unless>
+      <xacro:if value="${joint_limited}">
+        <limit lower="${-pi}" upper="${pi}" effort="28.0" velocity="${225. / 180. * pi}"/>
       </xacro:if>
       <dynamics damping="0.0" friction="0.0"/>
@@ -220,8 +214,8 @@
       <axis xyz="0 1 0" />
       <xacro:unless value="${joint_limited}">
-        <limit lower="${-2.0 * pi}" upper="${2.0 * pi}" effort="28.0" velocity="3.2"/>
-      </xacro:unless>
-      <xacro:if value="${joint_limited}">
-        <limit lower="${-pi}" upper="${pi}" effort="28.0" velocity="3.2"/>
+        <limit lower="${-180. / 180. * pi}" upper="${180. / 180. * pi}" effort="28.0" velocity="${225. / 180. * pi}"/>
+      </xacro:unless>
+      <xacro:if value="${joint_limited}">
+        <limit lower="${-pi}" upper="${pi}" effort="28.0" velocity="${225. / 180. * pi}"/>
       </xacro:if>
       <dynamics damping="0.0" friction="0.0"/>
@@ -230,5 +224,10 @@
       <visual>
         <geometry>
-	  <mesh filename="package://tm_description/meshes/tm700/visual/Wrist3.STL" />
+          <xacro:if value="${has_camera}">
+          <mesh filename="package://tm_description/meshes/tm700/visual/Wrist3.STL" />
+          </xacro:if>
+          <xacro:unless value="${has_camera}">
+          <mesh filename="package://tm_description/meshes/tm700/visual/Wrist3_no_camera.STL" />
+          </xacro:unless>
         </geometry>
 	<origin xyz="0 0 0.015" rpy="0 0 0"/>
@@ -239,5 +238,10 @@
       <collision>
         <geometry>
-	  <mesh filename="package://tm_description/meshes/tm700/collision/wrist_3.STL" />
+          <xacro:if value="${has_camera}">
+	      <mesh filename="package://tm_description/meshes/tm700/collision/wrist_3.STL" />
+          </xacro:if>
+          <xacro:unless value="${has_camera}">
+	      <mesh filename="package://tm_description/meshes/tm700/collision/wrist_3_no_camera.STL" />
+          </xacro:unless>
         </geometry>
       </collision>
@@ -252,8 +256,8 @@
       <axis xyz="0 0 1" />
       <xacro:unless value="${joint_limited}">
-        <limit lower="${-2.0 * pi}" upper="${2.0 * pi}" effort="28.0" velocity="3.2"/>
-      </xacro:unless>
-      <xacro:if value="${joint_limited}">
-        <limit lower="${-pi}" upper="${pi}" effort="28.0" velocity="3.2"/>
+        <limit lower="${-270. / 180. * pi}" upper="${270. / 180. * pi}" effort="28.0" velocity="${225. / 180. * pi}"/>
+      </xacro:unless>
+      <xacro:if value="${joint_limited}">
+        <limit lower="${-pi}" upper="${pi}" effort="28.0" velocity="${225. / 180. * pi}"/>
       </xacro:if>
       <dynamics damping="0.0" friction="0.0"/>
@@ -276,6 +280,6 @@
     <joint name="${prefix}base-base_link" type="fixed">
       <origin xyz="0 0 0" rpy="0 0 0"/>
-      <parent link="${prefix}base"/>
-      <child link="${prefix}base_link"/>
+      <parent link="${prefix}base_link"/>
+      <child link="${prefix}base"/>
     </joint>
     <!-- Frame coincident with all-zeros TCP on TM controller -->

File: tm_description/urdf/tm700_robot.urdf.xacro (robot description, xacro)
@@ -8,9 +8,9 @@
   <!-- tm700 -->
   <xacro:include filename="$(find tm_description)/urdf/tm700.urdf.xacro" />
-  <xacro:tm700_robot prefix="${prefix}" joint_limited="false" />
+  <xacro:tm700_robot prefix="${prefix}" joint_limited="false" has_camera="true" />
   <link name="world" />
   <joint name="world_joint" type="fixed">
     <parent link="world" />
-    <child link="base" />
+    <child link="base_link" />
     <origin xyz="0 0 0" rpy="0 0 0" />
   </joint>

File: tm_description/urdf/tm700_robot_eih.urdf.xacro (robot description, xacro)
@@ -8,9 +8,9 @@
   <!-- tm700 -->
   <xacro:include filename="$(find tm_description)/urdf/tm700.urdf.xacro" />
-  <xacro:tm700_robot prefix="${prefix}" joint_limited="false" />
+  <xacro:tm700_robot prefix="${prefix}" joint_limited="false" has_camera="true" />
   <link name="world" />
   <joint name="world_joint" type="fixed">
     <parent link="world" />
-    <child link="base" />
+    <child link="base_link" />
     <origin xyz="0 0 0" rpy="0 0 0" />
   </joint>

File: tm_description/urdf/tm700_robot_joint_limited.urdf.xacro (robot description, xacro)
@@ -8,9 +8,9 @@
   <!-- tm700 -->
   <xacro:include filename="$(find tm_description)/urdf/tm700.urdf.xacro" />
-  <xacro:tm700_robot prefix="${prefix}" joint_limited="true" />
+  <xacro:tm700_robot prefix="${prefix}" joint_limited="true" has_camera="true"/>
   <link name="world" />
   <joint name="world_joint" type="fixed">
     <parent link="world" />
-    <child link="base" />
+    <child link="base_link" />
     <origin xyz="0 0 0" rpy="0 0 0" />
   </joint>
